Commit message: feat: urdf ok

File: trc2026_description/urdf/trc2026.xacro (robot description, xacro)
@@ -24,5 +24,5 @@
   </collision>
 </link>
-<link name="wheel_right_forward_link_1">
+<link name="wheel_right_forward_link">
   <inertial>
     <origin xyz="6.208906921600921e-06 -0.03392279680272886 2.665693084685783e-06" rpy="0 0 0"/>
@@ -33,5 +33,5 @@
     <origin xyz="-0.4 0.257 0.1587" rpy="0 0 0"/>
     <geometry>
-      <mesh filename="file://$(find trc2026_description)/meshes/wheel_right_forward_link_1.stl" scale="0.001 0.001 0.001"/>
+      <mesh filename="file://$(find trc2026_description)/meshes/wheel_right_forward_link.stl" scale="0.001 0.001 0.001"/>
     </geometry>
     <material name="silver"/>
@@ -40,9 +40,9 @@
     <origin xyz="-0.4 0.257 0.1587" rpy="0 0 0"/>
     <geometry>
-      <mesh filename="file://$(find trc2026_description)/meshes/wheel_right_forward_link_1.stl" scale="0.001 0.001 0.001"/>
-    </geometry>
-  </collision>
-</link>
-<link name="steer_right_forward_link_1">
+      <mesh filename="file://$(find trc2026_description)/meshes/wheel_right_forward_link.stl" scale="0.001 0.001 0.001"/>
+    </geometry>
+  </collision>
+</link>
+<link name="steer_right_forward_link">
   <inertial>
     <origin xyz="9.4892602410801e-05 0.0606495493514779 -0.1482898116924078" rpy="0 0 0"/>
@@ -53,5 +53,5 @@
     <origin xyz="-0.4 0.292 -0.0646" rpy="0 0 0"/>
     <geometry>
-      <mesh filename="file://$(find trc2026_description)/meshes/steer_right_forward_link_1.stl" scale="0.001 0.001 0.001"/>
+      <mesh filename="file://$(find trc2026_description)/meshes/steer_right_forward_link.stl" scale="0.001 0.001 0.001"/>
     </geometry>
     <material name="silver"/>
@@ -60,9 +60,9 @@
     <origin xyz="-0.4 0.292 -0.0646" rpy="0 0 0"/>
     <geometry>
-      <mesh filename="file://$(find trc2026_description)/meshes/steer_right_forward_link_1.stl" scale="0.001 0.001 0.001"/>
-    </geometry>
-  </collision>
-</link>
-<link name="wheel_right_backward_link_1">
+      <mesh filename="file://$(find trc2026_description)/meshes/steer_right_forward_link.stl" scale="0.001 0.001 0.001"/>
+    </geometry>
+  </collision>
+</link>
+<link name="wheel_right_backward_link">
   <inertial>
     <origin xyz="-6.264940802247487e-06 -0.03392278637457424 -2.5014684090218786e-06" rpy="0 0 0"/>
@@ -73,5 +73,5 @@
     <origin xyz="0.4 0.257 0.1587" rpy="0 0 0"/>
     <geometry>
-      <mesh filename="file://$(find trc2026_description)/meshes/wheel_right_backward_link_1.stl" scale="0.001 0.001 0.001"/>
+      <mesh filename="file://$(find trc2026_description)/meshes/wheel_right_backward_link.stl" scale="0.001 0.001 0.001"/>
     </geometry>
     <material name="silver"/>
@@ -80,9 +80,9 @@
     <origin xyz="0.4 0.257 0.1587" rpy="0 0 0"/>
     <geometry>
-      <mesh filename="file://$(find trc2026_description)/meshes/wheel_right_backward_link_1.stl" scale="0.001 0.001 0.001"/>
-    </geometry>
-  </collision>
-</link>
-<link name="steer_right_backward_link_1">
+      <mesh filename="file://$(find trc2026_description)/meshes/wheel_right_backward_link.stl" scale="0.001 0.001 0.001"/>
+    </geometry>
+  </collision>
+</link>
+<link name="steer_right_backward_link">
   <inertial>
     <origin xyz="-9.48930291901906e-05 0.06064954512696477 -0.1482898108097947" rpy="0 0 0"/>
@@ -93,5 +93,5 @@
     <origin xyz="0.4 0.292 -0.0646" rpy="0 0 0"/>
     <geometry>
-      <mesh filename="file://$(find trc2026_description)/meshes/steer_right_backward_link_1.stl" scale="0.001 0.001 0.001"/>
+      <mesh filename="file://$(find trc2026_description)/meshes/steer_right_backward_link.stl" scale="0.001 0.001 0.001"/>
     </geometry>
     <material name="silver"/>
@@ -100,9 +100,9 @@
     <origin xyz="0.4 0.292 -0.0646" rpy="0 0 0"/>
     <geometry>
-      <mesh filename="file://$(find trc2026_description)/meshes/steer_right_backward_link_1.stl" scale="0.001 0.001 0.001"/>
-    </geometry>
-  </collision>
-</link>
-<link name="arm_right_link_1">
+      <mesh filename="file://$(find trc2026_description)/meshes/steer_right_backward_link.stl" scale="0.001 0.001 0.001"/>
+    </geometry>
+  </collision>
+</link>
+<link name="arm_right_link">
   <inertial>
     <origin xyz="-0.00014528539680006377 -0.22752633452724644 0.0012918534070657656" rpy="0 0 0"/>
@@ -113,5 +113,5 @@
     <origin xyz="0.0 0.036 -0.041" rpy="0 0 0"/>
     <geometry>
-      <mesh filename="file://$(find trc2026_description)/meshes/arm_right_link_1.stl" scale="0.001 0.001 0.001"/>
+      <mesh filename="file://$(find trc2026_description)/meshes/arm_right_link.stl" scale="0.001 0.001 0.001"/>
     </geometry>
     <material name="silver"/>
@@ -120,9 +120,9 @@
     <origin xyz="0.0 0.036 -0.041" rpy="0 0 0"/>
     <geometry>
-      <mesh filename="file://$(find trc2026_description)/meshes/arm_right_link_1.stl" scale="0.001 0.001 0.001"/>
-    </geometry>
-  </collision>
-</link>
-<link name="wheel_left_forward_link_1">
+      <mesh filename="file://$(find trc2026_description)/meshes/arm_right_link.stl" scale="0.001 0.001 0.001"/>
+    </geometry>
+  </collision>
+</link>
+<link name="wheel_left_forward_link">
   <inertial>
     <origin xyz="6.264940837497068e-06 0.03392278637456081 -2.501468379573213e-06" rpy="0 0 0"/>
@@ -133,5 +133,5 @@
     <origin xyz="-0.4 -0.257 0.1587" rpy="0 0 0"/>
     <geometry>
-      <mesh filename="file://$(find trc2026_description)/meshes/wheel_left_forward_link_1.stl" scale="0.001 0.001 0.001"/>
+      <mesh filename="file://$(find trc2026_description)/meshes/wheel_left_forward_link.stl" scale="0.001 0.001 0.001"/>
     </geometry>
     <material name="silver"/>
@@ -140,9 +140,9 @@
     <origin xyz="-0.4 -0.257 0.1587" rpy="0 0 0"/>
     <geometry>
-      <mesh filename="file://$(find trc2026_description)/meshes/wheel_left_forward_link_1.stl" scale="0.001 0.001 0.001"/>
-    </geometry>
-  </collision>
-</link>
-<link name="steer_left_forward_link_1">
+      <mesh filename="file://$(find trc2026_description)/meshes/wheel_left_forward_link.stl" scale="0.001 0.001 0.001"/>
+    </geometry>
+  </collision>
+</link>
+<link name="steer_left_forward_link">
   <inertial>
     <origin xyz="9.48930291901906e-05 0.5233504548730352 -0.019689810809794678" rpy="0 0 0"/>
@@ -151,18 +151,18 @@
   </inertial>
   <visual>
-    <origin xyz="-0.4 0.292 0.064" rpy="0 0 0"/>
-    <geometry>
-      <mesh filename="file://$(find trc2026_description)/meshes/steer_left_forward_link_1.stl" scale="0.001 0.001 0.001"/>
-    </geometry>
-    <material name="silver"/>
-  </visual>
-  <collision>
-    <origin xyz="-0.4 0.292 0.064" rpy="0 0 0"/>
-    <geometry>
-      <mesh filename="file://$(find trc2026_description)/meshes/steer_left_forward_link_1.stl" scale="0.001 0.001 0.001"/>
-    </geometry>
-  </collision>
-</link>
-<link name="wheel_left_backward_link_1">
+    <origin xyz="-0.4 -0.292 -0.064" rpy="0 0 0"/>
+    <geometry>
+      <mesh filename="file://$(find trc2026_description)/meshes/steer_left_forward_link.stl" scale="0.001 0.001 0.001"/>
+    </geometry>
+    <material name="silver"/>
+  </visual>
+  <collision>
+    <origin xyz="-0.4 -0.292 -0.064" rpy="0 0 0"/>
+    <geometry>
+      <mesh filename="file://$(find trc2026_description)/meshes/steer_left_forward_link.stl" scale="0.001 0.001 0.001"/>
+    </geometry>
+  </collision>
+</link>
+<link name="wheel_left_backward_link">
   <inertial>
     <origin xyz="-6.275711124770211e-06 0.03392279680272897 -2.5056050398652996e-06" rpy="0 0 0"/>
@@ -173,5 +173,5 @@
     <origin xyz="0.4 -0.257 0.1587" rpy="0 0 0"/>
     <geometry>
-      <mesh filename="file://$(find trc2026_description)/meshes/wheel_left_backward_link_1.stl" scale="0.001 0.001 0.001"/>
+      <mesh filename="file://$(find trc2026_description)/meshes/wheel_left_backward_link.stl" scale="0.001 0.001 0.001"/>
     </geometry>
     <material name="silver"/>
@@ -180,9 +180,9 @@
     <origin xyz="0.4 -0.257 0.1587" rpy="0 0 0"/>
     <geometry>
-      <mesh filename="file://$(find trc2026_description)/meshes/wheel_left_backward_link_1.stl" scale="0.001 0.001 0.001"/>
-    </geometry>
-  </collision>
-</link>
-<link name="steer_left_backward_link_1">
+      <mesh filename="file://$(find trc2026_description)/meshes/wheel_left_backward_link.stl" scale="0.001 0.001 0.001"/>
+    </geometry>
+  </collision>
+</link>
+<link name="steer_left_backward_link">
   <inertial>
     <origin xyz="-9.489260241096753e-05 0.5233504506485226 -0.019689811692407758" rpy="0 0 0"/>
@@ -191,18 +191,18 @@
   </inertial>
   <visual>
-    <origin xyz="0.4 0.292 0.064" rpy="0 0 0"/>
-    <geometry>
-      <mesh filename="file://$(find trc2026_description)/meshes/steer_left_backward_link_1.stl" scale="0.001 0.001 0.001"/>
-    </geometry>
-    <material name="silver"/>
-  </visual>
-  <collision>
-    <origin xyz="0.4 0.292 0.064" rpy="0 0 0"/>
-    <geometry>
-      <mesh filename="file://$(find trc2026_description)/meshes/steer_left_backward_link_1.stl" scale="0.001 0.001 0.001"/>
-    </geometry>
-  </collision>
-</link>
-<link name="arm_left_link_1">
+    <origin xyz="0.4 -0.292 -0.064" rpy="0 0 0"/>
+    <geometry>
+      <mesh filename="file://$(find trc2026_description)/meshes/steer_left_backward_link.stl" scale="0.001 0.001 0.001"/>
+    </geometry>
+    <material name="silver"/>
+  </visual>
+  <collision>
+    <origin xyz="0.4 -0.292 -0.064" rpy="0 0 0"/>
+    <geometry>
+      <mesh filename="file://$(find trc2026_description)/meshes/steer_left_backward_link.stl" scale="0.001 0.001 0.001"/>
+    </geometry>
+  </collision>
+</link>
+<link name="arm_left_link">
   <inertial>
     <origin xyz="-0.00014528539611865262 0.22752633467722524 0.0012918534957305841" rpy="0 0 0"/>
@@ -213,5 +213,5 @@
     <origin xyz="0.0 -0.036 -0.041" rpy="0 0 0"/>
     <geometry>
-      <mesh filename="file://$(find trc2026_description)/meshes/arm_left_link_1.stl" scale="0.001 0.001 0.001"/>
+      <mesh filename="file://$(find trc2026_description)/meshes/arm_left_link.stl" scale="0.001 0.001 0.001"/>
     </geometry>
     <material name="silver"/>
@@ -220,5 +220,5 @@
     <origin xyz="0.0 -0.036 -0.041" rpy="0 0 0"/>
     <geometry>
-      <mesh filename="file://$(find trc2026_description)/meshes/arm_left_link_1.stl" scale="0.001 0.001 0.001"/>
+      <mesh filename="file://$(find trc2026_description)/meshes/arm_left_link.stl" scale="0.001 0.001 0.001"/>
     </geometry>
   </collision>
@@ -226,24 +226,24 @@
 <joint name="回転 5" type="continuous">
   <origin xyz="0.0 0.035 -0.2233" rpy="0 0 0"/>
-  <parent link="steer_right_forward_link_1"/>
-  <child link="wheel_right_forward_link_1"/>
+  <parent link="steer_right_forward_link"/>
+  <child link="wheel_right_forward_link"/>
   <axis xyz="-0.0 1.0 -0.0"/>
 </joint>
 <joint name="回転 8" type="continuous">
   <origin xyz="0.4 -0.256 0.0236" rpy="0 0 0"/>
-  <parent link="arm_right_link_1"/>
-  <child link="steer_right_forward_link_1"/>
+  <parent link="arm_right_link"/>
+  <child link="steer_right_forward_link"/>
   <axis xyz="-0.0 0.0 -1.0"/>
 </joint>
 <joint name="回転 9" type="continuous">
   <origin xyz="0.0 0.035 -0.2233" rpy="0 0 0"/>
-  <parent link="steer_right_backward_link_1"/>
-  <child link="wheel_right_backward_link_1"/>
+  <parent link="steer_right_backward_link"/>
+  <child link="wheel_right_backward_link"/>
   <axis xyz="-0.0 -1.0 0.0"/>
 </joint>
 <joint name="回転 10" type="continuous">
   <origin xyz="-0.4 -0.256 0.0236" rpy="0 0 0"/>
-  <parent link="arm_right_link_1"/>
-  <child link="steer_right_backward_link_1"/>
+  <parent link="arm_right_link"/>
+  <child link="steer_right_backward_link"/>
   <axis xyz="0.0 -0.0 1.0"/>
 </joint>
@@ -251,29 +251,29 @@
   <origin xyz="0.0 -0.036 0.041" rpy="0 0 0"/>
   <parent link="base_link"/>
-  <child link="arm_right_link_1"/>
+  <child link="arm_right_link"/>
   <axis xyz="0.0 1.0 0.0"/>
 </joint>
 <joint name="回転 12" type="continuous">
-  <origin xyz="0.0 0.549 -0.0947" rpy="0 0 0"/>
-  <parent link="steer_left_forward_link_1"/>
-  <child link="wheel_left_forward_link_1"/>
+  <origin xyz="0.0 -0.035 -0.2233" rpy="0 0 0"/>
+  <parent link="steer_left_forward_link"/>
+  <child link="wheel_left_forward_link"/>
   <axis xyz="0.0 1.0 0.0"/>
 </joint>
 <joint name="回転 13" type="continuous">
-  <origin xyz="0.4 -0.328 -0.105" rpy="0 0 0"/>
-  <parent link="arm_left_link_1"/>
-  <child link="steer_left_forward_link_1"/>
+  <origin xyz="0.4 0.256 0.0236" rpy="0 0 0"/>
+  <parent link="arm_left_link"/>
+  <child link="steer_left_forward_link"/>
   <axis xyz="0.0 0.0 1.0"/>
 </joint>
 <joint name="回転 14" type="continuous">
-  <origin xyz="0.0 0.549 -0.0947" rpy="0 0 0"/>
-  <parent link="steer_left_backward_link_1"/>
-  <child link="wheel_left_backward_link_1"/>
+  <origin xyz="0.0 -0.035 -0.2233" rpy="0 0 0"/>
+  <parent link="steer_left_backward_link"/>
+  <child link="wheel_left_backward_link"/>
   <axis xyz="0.0 -1.0 -0.0"/>
 </joint>
 <joint name="回転 15" type="continuous">
-  <origin xyz="-0.4 -0.328 -0.105" rpy="0 0 0"/>
-  <parent link="arm_left_link_1"/>
-  <child link="steer_left_backward_link_1"/>
+  <origin xyz="-0.4 0.256 0.0236" rpy="0 0 0"/>
+  <parent link="arm_left_link"/>
+  <child link="steer_left_backward_link"/>
   <axis xyz="-0.0 -0.0 -1.0"/>
 </joint>
@@ -281,5 +281,5 @@
   <origin xyz="0.0 0.036 0.041" rpy="0 0 0"/>
   <parent link="base_link"/>
-  <child link="arm_left_link_1"/>
+  <child link="arm_left_link"/>
   <axis xyz="-0.0 1.0 -0.0"/>
 </joint>

Commit message: feat: gazebo launch

File: trc2026_description/urdf/trc2026.xacro (robot description, xacro)
@@ -224,5 +224,5 @@
   </collision>
 </link>
-<joint name="回転 5" type="continuous">
+<joint name="drive_right_forward_joint" type="continuous">
   <origin xyz="0.0 0.035 -0.2233" rpy="0 0 0"/>
   <parent link="steer_right_forward_link"/>
@@ -230,5 +230,5 @@
   <axis xyz="-0.0 1.0 -0.0"/>
 </joint>
-<joint name="回転 8" type="continuous">
+<joint name="steer_right_forward_joint" type="continuous">
   <origin xyz="0.4 -0.256 0.0236" rpy="0 0 0"/>
   <parent link="arm_right_link"/>
@@ -236,5 +236,5 @@
   <axis xyz="-0.0 0.0 -1.0"/>
 </joint>
-<joint name="回転 9" type="continuous">
+<joint name="drive_right_backward_joint" type="continuous">
   <origin xyz="0.0 0.035 -0.2233" rpy="0 0 0"/>
   <parent link="steer_right_backward_link"/>
@@ -242,5 +242,5 @@
   <axis xyz="-0.0 -1.0 0.0"/>
 </joint>
-<joint name="回転 10" type="continuous">
+<joint name="steer_right_backward_joint" type="continuous">
   <origin xyz="-0.4 -0.256 0.0236" rpy="0 0 0"/>
   <parent link="arm_right_link"/>
@@ -248,5 +248,5 @@
   <axis xyz="0.0 -0.0 1.0"/>
 </joint>
-<joint name="回転 11" type="continuous">
+<joint name="arm_right_joint" type="fixed">
   <origin xyz="0.0 -0.036 0.041" rpy="0 0 0"/>
   <parent link="base_link"/>
@@ -254,5 +254,5 @@
   <axis xyz="0.0 1.0 0.0"/>
 </joint>
-<joint name="回転 12" type="continuous">
+<joint name="drive_left_forward_joint" type="continuous">
   <origin xyz="0.0 -0.035 -0.2233" rpy="0 0 0"/>
   <parent link="steer_left_forward_link"/>
@@ -260,5 +260,5 @@
   <axis xyz="0.0 1.0 0.0"/>
 </joint>
-<joint name="回転 13" type="continuous">
+<joint name="steer_left_forward_joint" type="continuous">
   <origin xyz="0.4 0.256 0.0236" rpy="0 0 0"/>
   <parent link="arm_left_link"/>
@@ -266,5 +266,5 @@
   <axis xyz="0.0 0.0 1.0"/>
 </joint>
-<joint name="回転 14" type="continuous">
+<joint name="drive_left_backward_joint" type="continuous">
   <origin xyz="0.0 -0.035 -0.2233" rpy="0 0 0"/>
   <parent link="steer_left_backward_link"/>
@@ -272,5 +272,5 @@
   <axis xyz="0.0 -1.0 -0.0"/>
 </joint>
-<joint name="回転 15" type="continuous">
+<joint name="steer_left_backward_joint" type="continuous">
   <origin xyz="-0.4 0.256 0.0236" rpy="0 0 0"/>
   <parent link="arm_left_link"/>
@@ -278,5 +278,5 @@
   <axis xyz="-0.0 -0.0 -1.0"/>
 </joint>
-<joint name="回転 16" type="continuous">
+<joint name="arm_left_joint" type="fixed">
   <origin xyz="0.0 0.036 0.041" rpy="0 0 0"/>
   <parent link="base_link"/>

Commit message: feat: add gazebo sensors

File: trc2026_description/urdf/trc2026.xacro (robot description, xacro)
@@ -224,4 +224,25 @@
   </collision>
 </link>
+<link name="base_scan">
+    <inertial>
+        <origin xyz="0 0 4" rpy="0 0 0"/>
+        <mass value="0.1"/>
+        <inertia ixx="1e-6" ixy="0" ixz="0" iyy="1e-6" iyz="0" izz="1e-6"/>
+    </inertial>
+</link>
+<link name="imu_link">
+  <inertial>
+    <mass value="0.01"/>
+    <origin xyz="0 0 0" rpy="0 0 0"/>
+    <inertia ixx="1e-6" ixy="0" ixz="0" iyy="1e-6" iyz="0" izz="1e-6"/>
+  </inertial>
+</link>
+<link name="camera_link">
+  <inertial>
+    <mass value="0.01"/>
+    <origin xyz="0 0 0" rpy="0 0 0"/>
+    <inertia ixx="1e-6" ixy="0" ixz="0" iyy="1e-6" iyz="0" izz="1e-6"/>
+  </inertial>
+</link>
 <joint name="drive_right_forward_joint" type="continuous">
   <origin xyz="0.0 0.035 -0.2233" rpy="0 0 0"/>
@@ -284,3 +305,18 @@
   <axis xyz="-0.0 1.0 -0.0"/>
 </joint>
+<joint name="imu_joint" type="fixed">
+    <parent link="base_link"/>
+    <child link="imu_link"/>
+    <origin xyz="-0.05 0 0.08" rpy="0 0 0"/>
+</joint>
+<joint name="lidar_joint" type="fixed">
+    <parent link="base_link"/>
+    <child link="base_scan"/>
+    <origin xyz="0.055 0 0.13" rpy="0 0 0"/>
+</joint>
+<joint name="camera_joint" type="fixed">
+    <parent link="base_link"/>
+    <child link="camera_link"/>
+    <origin xyz="0.1 0 0.15" rpy="0 0 0"/>
+</joint>
 </robot>

Commit message: feat: integrate nav2

File: trc2026_description/urdf/trc2026.xacro (robot description, xacro)
@@ -4,4 +4,10 @@
 <xacro:include filename="$(find trc2026_description)/urdf/trc2026.trans" />
 <xacro:include filename="$(find trc2026_description)/urdf/trc2026.gazebo" />
+<link name="base_footprint"/>
+<joint name="base_link_joint" type="fixed">
+  <parent link="base_footprint"/>
+  <child link="base_link"/>
+  <origin xyz="0 0 0.30" rpy="0 0 0"/>
+ </joint>
 <link name="base_link">
   <inertial>
@@ -226,5 +232,5 @@
 <link name="base_scan">
     <inertial>
-        <origin xyz="0 0 4" rpy="0 0 0"/>
+        <origin xyz="0 0 0" rpy="0 0 0"/>
         <mass value="0.1"/>
         <inertia ixx="1e-6" ixy="0" ixz="0" iyy="1e-6" iyz="0" izz="1e-6"/>
@@ -313,5 +319,5 @@
     <parent link="base_link"/>
     <child link="base_scan"/>
-    <origin xyz="0.055 0 0.13" rpy="0 0 0"/>
+    <origin xyz="0.055 0 0.2" rpy="0 0 0"/>
 </joint>
 <joint name="camera_joint" type="fixed">
