Commit message: feat: urdf display ok

File: trc2026_description/urdf/trc2026.xacro (robot description, xacro)
@@ -19,5 +19,5 @@
     <origin xyz="0 0 0" rpy="0 0 0"/>
     <geometry>
-      <mesh filename="file://$(find trc2026_description)/meshes/base_link.stl" scale="0.001 0.001 0.001"/>
+      <mesh filename="package://trc2026_description/meshes/base_link.stl" scale="0.001 0.001 0.001"/>
     </geometry>
     <material name="silver"/>
@@ -26,5 +26,5 @@
     <origin xyz="0 0 0" rpy="0 0 0"/>
     <geometry>
-      <mesh filename="file://$(find trc2026_description)/meshes/base_link.stl" scale="0.001 0.001 0.001"/>
+      <mesh filename="package://trc2026_description/meshes/base_link.stl" scale="0.001 0.001 0.001"/>
     </geometry>
   </collision>
@@ -39,5 +39,5 @@
     <origin xyz="-0.4 0.257 0.1587" rpy="0 0 0"/>
     <geometry>
-      <mesh filename="file://$(find trc2026_description)/meshes/wheel_right_forward_link.stl" scale="0.001 0.001 0.001"/>
+      <mesh filename="package://trc2026_description/meshes/wheel_right_forward_link.stl" scale="0.001 0.001 0.001"/>
     </geometry>
     <material name="silver"/>
@@ -46,5 +46,5 @@
     <origin xyz="-0.4 0.257 0.1587" rpy="0 0 0"/>
     <geometry>
-      <mesh filename="file://$(find trc2026_description)/meshes/wheel_right_forward_link.stl" scale="0.001 0.001 0.001"/>
+      <mesh filename="package://trc2026_description/meshes/wheel_right_forward_link.stl" scale="0.001 0.001 0.001"/>
     </geometry>
   </collision>
@@ -59,5 +59,5 @@
     <origin xyz="-0.4 0.292 -0.0646" rpy="0 0 0"/>
     <geometry>
-      <mesh filename="file://$(find trc2026_description)/meshes/steer_right_forward_link.stl" scale="0.001 0.001 0.001"/>
+      <mesh filename="package://trc2026_description/meshes/steer_right_forward_link.stl" scale="0.001 0.001 0.001"/>
     </geometry>
     <material name="silver"/>
@@ -66,5 +66,5 @@
     <origin xyz="-0.4 0.292 -0.0646" rpy="0 0 0"/>
     <geometry>
-      <mesh filename="file://$(find trc2026_description)/meshes/steer_right_forward_link.stl" scale="0.001 0.001 0.001"/>
+      <mesh filename="package://trc2026_description/meshes/steer_right_forward_link.stl" scale="0.001 0.001 0.001"/>
     </geometry>
   </collision>
@@ -79,5 +79,5 @@
     <origin xyz="0.4 0.257 0.1587" rpy="0 0 0"/>
     <geometry>
-      <mesh filename="file://$(find trc2026_description)/meshes/wheel_right_backward_link.stl" scale="0.001 0.001 0.001"/>
+      <mesh filename="package://trc2026_description/meshes/wheel_right_backward_link.stl" scale="0.001 0.001 0.001"/>
     </geometry>
     <material name="silver"/>
@@ -86,5 +86,5 @@
     <origin xyz="0.4 0.257 0.1587" rpy="0 0 0"/>
     <geometry>
-      <mesh filename="file://$(find trc2026_description)/meshes/wheel_right_backward_link.stl" scale="0.001 0.001 0.001"/>
+      <mesh filename="package://trc2026_description/meshes/wheel_right_backward_link.stl" scale="0.001 0.001 0.001"/>
     </geometry>
   </collision>
@@ -99,5 +99,5 @@
     <origin xyz="0.4 0.292 -0.0646" rpy="0 0 0"/>
     <geometry>
-      <mesh filename="file://$(find trc2026_description)/meshes/steer_right_backward_link.stl" scale="0.001 0.001 0.001"/>
+      <mesh filename="package://trc2026_description/meshes/steer_right_backward_link.stl" scale="0.001 0.001 0.001"/>
     </geometry>
     <material name="silver"/>
@@ -106,5 +106,5 @@
     <origin xyz="0.4 0.292 -0.0646" rpy="0 0 0"/>
     <geometry>
-      <mesh filename="file://$(find trc2026_description)/meshes/steer_right_backward_link.stl" scale="0.001 0.001 0.001"/>
+      <mesh filename="package://trc2026_description/meshes/steer_right_backward_link.stl" scale="0.001 0.001 0.001"/>
     </geometry>
   </collision>
@@ -119,5 +119,5 @@
     <origin xyz="0.0 0.036 -0.041" rpy="0 0 0"/>
     <geometry>
-      <mesh filename="file://$(find trc2026_description)/meshes/arm_right_link.stl" scale="0.001 0.001 0.001"/>
+      <mesh filename="package://trc2026_description/meshes/arm_right_link.stl" scale="0.001 0.001 0.001"/>
     </geometry>
     <material name="silver"/>
@@ -126,5 +126,5 @@
     <origin xyz="0.0 0.036 -0.041" rpy="0 0 0"/>
     <geometry>
-      <mesh filename="file://$(find trc2026_description)/meshes/arm_right_link.stl" scale="0.001 0.001 0.001"/>
+      <mesh filename="package://trc2026_description/meshes/arm_right_link.stl" scale="0.001 0.001 0.001"/>
     </geometry>
   </collision>
@@ -139,5 +139,5 @@
     <origin xyz="-0.4 -0.257 0.1587" rpy="0 0 0"/>
     <geometry>
-      <mesh filename="file://$(find trc2026_description)/meshes/wheel_left_forward_link.stl" scale="0.001 0.001 0.001"/>
+      <mesh filename="package://trc2026_description/meshes/wheel_left_forward_link.stl" scale="0.001 0.001 0.001"/>
     </geometry>
     <material name="silver"/>
@@ -146,5 +146,5 @@
     <origin xyz="-0.4 -0.257 0.1587" rpy="0 0 0"/>
     <geometry>
-      <mesh filename="file://$(find trc2026_description)/meshes/wheel_left_forward_link.stl" scale="0.001 0.001 0.001"/>
+      <mesh filename="package://trc2026_description/meshes/wheel_left_forward_link.stl" scale="0.001 0.001 0.001"/>
     </geometry>
   </collision>
@@ -159,5 +159,5 @@
     <origin xyz="-0.4 -0.292 -0.064" rpy="0 0 0"/>
     <geometry>
-      <mesh filename="file://$(find trc2026_description)/meshes/steer_left_forward_link.stl" scale="0.001 0.001 0.001"/>
+      <mesh filename="package://trc2026_description/meshes/steer_left_forward_link.stl" scale="0.001 0.001 0.001"/>
     </geometry>
     <material name="silver"/>
@@ -166,5 +166,5 @@
     <origin xyz="-0.4 -0.292 -0.064" rpy="0 0 0"/>
     <geometry>
-      <mesh filename="file://$(find trc2026_description)/meshes/steer_left_forward_link.stl" scale="0.001 0.001 0.001"/>
+      <mesh filename="package://trc2026_description/meshes/steer_left_forward_link.stl" scale="0.001 0.001 0.001"/>
     </geometry>
   </collision>
@@ -179,5 +179,5 @@
     <origin xyz="0.4 -0.257 0.1587" rpy="0 0 0"/>
     <geometry>
-      <mesh filename="file://$(find trc2026_description)/meshes/wheel_left_backward_link.stl" scale="0.001 0.001 0.001"/>
+      <mesh filename="package://trc2026_description/meshes/wheel_left_backward_link.stl" scale="0.001 0.001 0.001"/>
     </geometry>
     <material name="silver"/>
@@ -186,5 +186,5 @@
     <origin xyz="0.4 -0.257 0.1587" rpy="0 0 0"/>
     <geometry>
-      <mesh filename="file://$(find trc2026_description)/meshes/wheel_left_backward_link.stl" scale="0.001 0.001 0.001"/>
+      <mesh filename="package://trc2026_description/meshes/wheel_left_backward_link.stl" scale="0.001 0.001 0.001"/>
     </geometry>
   </collision>
@@ -199,5 +199,5 @@
     <origin xyz="0.4 -0.292 -0.064" rpy="0 0 0"/>
     <geometry>
-      <mesh filename="file://$(find trc2026_description)/meshes/steer_left_backward_link.stl" scale="0.001 0.001 0.001"/>
+      <mesh filename="package://trc2026_description/meshes/steer_left_backward_link.stl" scale="0.001 0.001 0.001"/>
     </geometry>
     <material name="silver"/>
@@ -206,5 +206,5 @@
     <origin xyz="0.4 -0.292 -0.064" rpy="0 0 0"/>
     <geometry>
-      <mesh filename="file://$(find trc2026_description)/meshes/steer_left_backward_link.stl" scale="0.001 0.001 0.001"/>
+      <mesh filename="package://trc2026_description/meshes/steer_left_backward_link.stl" scale="0.001 0.001 0.001"/>
     </geometry>
   </collision>
@@ -219,5 +219,5 @@
     <origin xyz="0.0 -0.036 -0.041" rpy="0 0 0"/>
     <geometry>
-      <mesh filename="file://$(find trc2026_description)/meshes/arm_left_link.stl" scale="0.001 0.001 0.001"/>
+      <mesh filename="package://trc2026_description/meshes/arm_left_link.stl" scale="0.001 0.001 0.001"/>
     </geometry>
     <material name="silver"/>
@@ -226,5 +226,5 @@
     <origin xyz="0.0 -0.036 -0.041" rpy="0 0 0"/>
     <geometry>
-      <mesh filename="file://$(find trc2026_description)/meshes/arm_left_link.stl" scale="0.001 0.001 0.001"/>
+      <mesh filename="package://trc2026_description/meshes/arm_left_link.stl" scale="0.001 0.001 0.001"/>
     </geometry>
   </collision>
