Commit message: feat: moveit worked

File: trc2026_description/urdf/trc2026.xacro (robot description, xacro)
@@ -2,4 +2,5 @@
 <robot name="trc2026"
   xmlns:xacro="http://www.ros.org/wiki/xacro">
+  <xacro:arg name="use_fake_hardware"            default="false" />
   <xacro:include filename="$(find trc2026_description)/urdf/materials.xacro" />
   <xacro:include filename="$(find trc2026_description)/urdf/trc2026.trans" />
@@ -240,12 +241,12 @@
       <origin xyz="0 0 0" rpy="0 0 0"/>
       <geometry>
-        <mesh filename="file://$(find trc2026_description)/meshes/arm_1_link.stl" scale="0.001 0.001 0.001"/>
-      </geometry>
-      <material name="silver"/>
-    </visual>
-    <collision>
-      <origin xyz="0 0 0" rpy="0 0 0"/>
-      <geometry>
-        <mesh filename="file://$(find trc2026_description)/meshes/arm_1_link.stl" scale="0.001 0.001 0.001"/>
+        <mesh filename="package://trc2026_description/meshes/arm_1_link.stl" scale="0.001 0.001 0.001"/>
+      </geometry>
+      <material name="silver"/>
+    </visual>
+    <collision>
+      <origin xyz="0 0 0" rpy="0 0 0"/>
+      <geometry>
+        <mesh filename="package://trc2026_description/meshes/arm_1_link.stl" scale="0.001 0.001 0.001"/>
       </geometry>
     </collision>
@@ -260,5 +261,5 @@
       <origin xyz="0.1077 -3e-06 -0.960058" rpy="0 0 0"/>
       <geometry>
-        <mesh filename="file://$(find trc2026_description)/meshes/hand_right_link.stl" scale="0.001 0.001 0.001"/>
+        <mesh filename="package://trc2026_description/meshes/hand_right_link.stl" scale="0.001 0.001 0.001"/>
       </geometry>
       <material name="silver"/>
@@ -267,5 +268,5 @@
       <origin xyz="0.1077 -3e-06 -0.960058" rpy="0 0 0"/>
       <geometry>
-        <mesh filename="file://$(find trc2026_description)/meshes/hand_right_link.stl" scale="0.001 0.001 0.001"/>
+        <mesh filename="package://trc2026_description/meshes/hand_right_link.stl" scale="0.001 0.001 0.001"/>
       </geometry>
     </collision>
@@ -280,5 +281,5 @@
       <origin xyz="-0.1077 -3e-06 -0.960058" rpy="0 0 0"/>
       <geometry>
-        <mesh filename="file://$(find trc2026_description)/meshes/hand_left_link.stl" scale="0.001 0.001 0.001"/>
+        <mesh filename="package://trc2026_description/meshes/hand_left_link.stl" scale="0.001 0.001 0.001"/>
       </geometry>
       <material name="silver"/>
@@ -287,5 +288,5 @@
       <origin xyz="-0.1077 -3e-06 -0.960058" rpy="0 0 0"/>
       <geometry>
-        <mesh filename="file://$(find trc2026_description)/meshes/hand_left_link.stl" scale="0.001 0.001 0.001"/>
+        <mesh filename="package://trc2026_description/meshes/hand_left_link.stl" scale="0.001 0.001 0.001"/>
       </geometry>
     </collision>
@@ -300,5 +301,5 @@
       <origin xyz="0 0 -0.882" rpy="0 0 0"/>
       <geometry>
-        <mesh filename="file://$(find trc2026_description)/meshes/arm_4_link.stl" scale="0.001 0.001 0.001"/>
+        <mesh filename="package://trc2026_description/meshes/arm_4_link.stl" scale="0.001 0.001 0.001"/>
       </geometry>
       <material name="silver"/>
@@ -307,5 +308,5 @@
       <origin xyz="0 0 -0.882" rpy="0 0 0"/>
       <geometry>
-        <mesh filename="file://$(find trc2026_description)/meshes/arm_4_link.stl" scale="0.001 0.001 0.001"/>
+        <mesh filename="package://trc2026_description/meshes/arm_4_link.stl" scale="0.001 0.001 0.001"/>
       </geometry>
     </collision>
@@ -320,5 +321,5 @@
       <origin xyz="0 0 -0.482" rpy="0 0 0"/>
       <geometry>
-        <mesh filename="file://$(find trc2026_description)/meshes/arm_3_link.stl" scale="0.001 0.001 0.001"/>
+        <mesh filename="package://trc2026_description/meshes/arm_3_link.stl" scale="0.001 0.001 0.001"/>
       </geometry>
       <material name="silver"/>
@@ -327,5 +328,5 @@
       <origin xyz="0 0 -0.482" rpy="0 0 0"/>
       <geometry>
-        <mesh filename="file://$(find trc2026_description)/meshes/arm_3_link.stl" scale="0.001 0.001 0.001"/>
+        <mesh filename="package://trc2026_description/meshes/arm_3_link.stl" scale="0.001 0.001 0.001"/>
       </geometry>
     </collision>
@@ -340,5 +341,5 @@
       <origin xyz="-0.056 -0.0 -0.082" rpy="0 0 0"/>
       <geometry>
-        <mesh filename="file://$(find trc2026_description)/meshes/arm_2_link.stl" scale="0.001 0.001 0.001"/>
+        <mesh filename="package://trc2026_description/meshes/arm_2_link.stl" scale="0.001 0.001 0.001"/>
       </geometry>
       <material name="silver"/>
@@ -347,5 +348,5 @@
       <origin xyz="-0.056 -0.0 -0.082" rpy="0 0 0"/>
       <geometry>
-        <mesh filename="file://$(find trc2026_description)/meshes/arm_2_link.stl" scale="0.001 0.001 0.001"/>
+        <mesh filename="package://trc2026_description/meshes/arm_2_link.stl" scale="0.001 0.001 0.001"/>
       </geometry>
     </collision>
@@ -360,5 +361,5 @@
       <origin xyz="0.0 0 -0.082" rpy="0 0 0"/>
       <geometry>
-        <mesh filename="file://$(find trc2026_description)/meshes/arm_3_rotate_link.stl" scale="0.001 0.001 0.001"/>
+        <mesh filename="package://trc2026_description/meshes/arm_3_rotate_link.stl" scale="0.001 0.001 0.001"/>
       </geometry>
       <material name="silver"/>
@@ -367,5 +368,5 @@
       <origin xyz="0.0 0 -0.082" rpy="0 0 0"/>
       <geometry>
-        <mesh filename="file://$(find trc2026_description)/meshes/arm_3_rotate_link.stl" scale="0.001 0.001 0.001"/>
+        <mesh filename="package://trc2026_description/meshes/arm_3_rotate_link.stl" scale="0.001 0.001 0.001"/>
       </geometry>
     </collision>
@@ -380,5 +381,5 @@
       <origin xyz="0.0 -0.099619 -0.090716" rpy="0 0 0"/>
       <geometry>
-        <mesh filename="file://$(find trc2026_description)/meshes/arm_3_shaft_link.stl" scale="0.001 0.001 0.001"/>
+        <mesh filename="package://trc2026_description/meshes/arm_3_shaft_link.stl" scale="0.001 0.001 0.001"/>
       </geometry>
       <material name="silver"/>
@@ -387,5 +388,5 @@
       <origin xyz="0.0 -0.099619 -0.090716" rpy="0 0 0"/>
       <geometry>
-        <mesh filename="file://$(find trc2026_description)/meshes/arm_3_shaft_link.stl" scale="0.001 0.001 0.001"/>
+        <mesh filename="package://trc2026_description/meshes/arm_3_shaft_link.stl" scale="0.001 0.001 0.001"/>
       </geometry>
     </collision>
@@ -413,5 +414,5 @@
       <inertia ixx="1e-6" ixy="0" ixz="0" iyy="1e-6" iyz="0" izz="1e-6"/>
     </inertial>
-  </link>>
+  </link>
   <joint name="drive_right_forward_joint" type="continuous">
     <origin xyz="0.0 0.035 -0.2233" rpy="0 0 0"/>
@@ -514,16 +515,16 @@
     <mimic joint="arm_2_joint" multiplier="-1.0" offset="0.0"/>
   </joint>
-  <joint name="arm_3_rotate_joint" type="continuous">
+  <joint name="arm_3_joint" type="continuous">
     <origin xyz="0 0 0" rpy="0 0 0"/>
     <parent link="arm_3_virtual_link"/>
     <child link="arm_3_link"/>
     <axis xyz="1.0 0.0 0.0"/>
-    <mimic joint="arm_3_joint" multiplier="1.0" offset="1.6"/>
-  </joint>
-  <joint name="arm_3_joint" type="continuous">
+  </joint>
+  <joint name="arm_3_motor_joint" type="continuous">
     <origin xyz="0.0 0 0.082" rpy="0 0 0"/>
     <parent link="arm_1_link"/>
     <child link="arm_3_rotate_link"/>
     <axis xyz="1.0 0.0 0.0"/>
+    <mimic joint="arm_3_joint" multiplier="1.0" offset="-1.6"/>
   </joint>
   <joint name="arm_3_joint_reversal" type="continuous">
@@ -532,5 +533,5 @@
     <child link="shaft_virtual_link"/>
     <axis xyz="1.0 0.0 0.0"/>
-    <mimic joint="arm_3_joint" multiplier="-1.0" offset="0.0"/>
+    <mimic joint="arm_3_motor_joint" multiplier="-1.0" offset="0.0"/>
   </joint>
   <joint name="arm_3_virtual_joint" type="continuous">

Commit message: fix: missing urdf

File: trc2026_description/urdf/trc2026.xacro (robot description, xacro)
@@ -240,12 +240,12 @@
       <origin xyz="0 0 0" rpy="0 0 0"/>
       <geometry>
-        <mesh filename="file://$(find trc2026_description)/meshes/arm_1_link.stl" scale="0.001 0.001 0.001"/>
-      </geometry>
-      <material name="silver"/>
-    </visual>
-    <collision>
-      <origin xyz="0 0 0" rpy="0 0 0"/>
-      <geometry>
-        <mesh filename="file://$(find trc2026_description)/meshes/arm_1_link.stl" scale="0.001 0.001 0.001"/>
+        <mesh filename="package://trc2026_description/meshes/arm_1_link.stl" scale="0.001 0.001 0.001"/>
+      </geometry>
+      <material name="silver"/>
+    </visual>
+    <collision>
+      <origin xyz="0 0 0" rpy="0 0 0"/>
+      <geometry>
+        <mesh filename="package://trc2026_description/meshes/arm_1_link.stl" scale="0.001 0.001 0.001"/>
       </geometry>
     </collision>
@@ -260,5 +260,5 @@
       <origin xyz="0.1077 -3e-06 -0.960058" rpy="0 0 0"/>
       <geometry>
-        <mesh filename="file://$(find trc2026_description)/meshes/hand_right_link.stl" scale="0.001 0.001 0.001"/>
+        <mesh filename="package://trc2026_description/meshes/hand_right_link.stl" scale="0.001 0.001 0.001"/>
       </geometry>
       <material name="silver"/>
@@ -267,5 +267,5 @@
       <origin xyz="0.1077 -3e-06 -0.960058" rpy="0 0 0"/>
       <geometry>
-        <mesh filename="file://$(find trc2026_description)/meshes/hand_right_link.stl" scale="0.001 0.001 0.001"/>
+        <mesh filename="package://trc2026_description/meshes/hand_right_link.stl" scale="0.001 0.001 0.001"/>
       </geometry>
     </collision>
@@ -280,5 +280,5 @@
       <origin xyz="-0.1077 -3e-06 -0.960058" rpy="0 0 0"/>
       <geometry>
-        <mesh filename="file://$(find trc2026_description)/meshes/hand_left_link.stl" scale="0.001 0.001 0.001"/>
+        <mesh filename="package://trc2026_description/meshes/hand_left_link.stl" scale="0.001 0.001 0.001"/>
       </geometry>
       <material name="silver"/>
@@ -287,5 +287,5 @@
       <origin xyz="-0.1077 -3e-06 -0.960058" rpy="0 0 0"/>
       <geometry>
-        <mesh filename="file://$(find trc2026_description)/meshes/hand_left_link.stl" scale="0.001 0.001 0.001"/>
+        <mesh filename="package://trc2026_description/meshes/hand_left_link.stl" scale="0.001 0.001 0.001"/>
       </geometry>
     </collision>
@@ -300,5 +300,5 @@
       <origin xyz="0 0 -0.882" rpy="0 0 0"/>
       <geometry>
-        <mesh filename="file://$(find trc2026_description)/meshes/arm_4_link.stl" scale="0.001 0.001 0.001"/>
+        <mesh filename="package://trc2026_description/meshes/arm_4_link.stl" scale="0.001 0.001 0.001"/>
       </geometry>
       <material name="silver"/>
@@ -307,5 +307,5 @@
       <origin xyz="0 0 -0.882" rpy="0 0 0"/>
       <geometry>
-        <mesh filename="file://$(find trc2026_description)/meshes/arm_4_link.stl" scale="0.001 0.001 0.001"/>
+        <mesh filename="package://trc2026_description/meshes/arm_4_link.stl" scale="0.001 0.001 0.001"/>
       </geometry>
     </collision>
@@ -320,5 +320,5 @@
       <origin xyz="0 0 -0.482" rpy="0 0 0"/>
       <geometry>
-        <mesh filename="file://$(find trc2026_description)/meshes/arm_3_link.stl" scale="0.001 0.001 0.001"/>
+        <mesh filename="package://trc2026_description/meshes/arm_3_link.stl" scale="0.001 0.001 0.001"/>
       </geometry>
       <material name="silver"/>
@@ -327,5 +327,5 @@
       <origin xyz="0 0 -0.482" rpy="0 0 0"/>
       <geometry>
-        <mesh filename="file://$(find trc2026_description)/meshes/arm_3_link.stl" scale="0.001 0.001 0.001"/>
+        <mesh filename="package://trc2026_description/meshes/arm_3_link.stl" scale="0.001 0.001 0.001"/>
       </geometry>
     </collision>
@@ -340,5 +340,5 @@
       <origin xyz="-0.056 -0.0 -0.082" rpy="0 0 0"/>
       <geometry>
-        <mesh filename="file://$(find trc2026_description)/meshes/arm_2_link.stl" scale="0.001 0.001 0.001"/>
+        <mesh filename="package://trc2026_description/meshes/arm_2_link.stl" scale="0.001 0.001 0.001"/>
       </geometry>
       <material name="silver"/>
@@ -347,5 +347,5 @@
       <origin xyz="-0.056 -0.0 -0.082" rpy="0 0 0"/>
       <geometry>
-        <mesh filename="file://$(find trc2026_description)/meshes/arm_2_link.stl" scale="0.001 0.001 0.001"/>
+        <mesh filename="package://trc2026_description/meshes/arm_2_link.stl" scale="0.001 0.001 0.001"/>
       </geometry>
     </collision>
@@ -360,5 +360,5 @@
       <origin xyz="0.0 0 -0.082" rpy="0 0 0"/>
       <geometry>
-        <mesh filename="file://$(find trc2026_description)/meshes/arm_3_rotate_link.stl" scale="0.001 0.001 0.001"/>
+        <mesh filename="package://trc2026_description/meshes/arm_3_rotate_link.stl" scale="0.001 0.001 0.001"/>
       </geometry>
       <material name="silver"/>
@@ -367,5 +367,5 @@
       <origin xyz="0.0 0 -0.082" rpy="0 0 0"/>
       <geometry>
-        <mesh filename="file://$(find trc2026_description)/meshes/arm_3_rotate_link.stl" scale="0.001 0.001 0.001"/>
+        <mesh filename="package://trc2026_description/meshes/arm_3_rotate_link.stl" scale="0.001 0.001 0.001"/>
       </geometry>
     </collision>
@@ -380,5 +380,5 @@
       <origin xyz="0.0 -0.099619 -0.090716" rpy="0 0 0"/>
       <geometry>
-        <mesh filename="file://$(find trc2026_description)/meshes/arm_3_shaft_link.stl" scale="0.001 0.001 0.001"/>
+        <mesh filename="package://trc2026_description/meshes/arm_3_shaft_link.stl" scale="0.001 0.001 0.001"/>
       </geometry>
       <material name="silver"/>
@@ -387,5 +387,5 @@
       <origin xyz="0.0 -0.099619 -0.090716" rpy="0 0 0"/>
       <geometry>
-        <mesh filename="file://$(find trc2026_description)/meshes/arm_3_shaft_link.stl" scale="0.001 0.001 0.001"/>
+        <mesh filename="package://trc2026_description/meshes/arm_3_shaft_link.stl" scale="0.001 0.001 0.001"/>
       </geometry>
     </collision>
@@ -413,5 +413,5 @@
       <inertia ixx="1e-6" ixy="0" ixz="0" iyy="1e-6" iyz="0" izz="1e-6"/>
     </inertial>
-  </link>>
+  </link>
   <joint name="drive_right_forward_joint" type="continuous">
     <origin xyz="0.0 0.035 -0.2233" rpy="0 0 0"/>

Commit message: feat: arucoマーカーの検出

File: trc2026_description/urdf/trc2026.xacro (robot description, xacro)
@@ -555,5 +555,5 @@
     <parent link="base_link"/>
     <child link="camera_link"/>
-    <origin xyz="0.1 0 0.15" rpy="0 0 0"/>
+    <origin xyz="0.3 0 0.10" rpy="0 0 0"/>
   </joint>
 </robot>

Commit message: chore: delete depth from AR marker recognition

File: trc2026_description/urdf/trc2026.xacro (robot description, xacro)
@@ -408,5 +408,5 @@
     </inertial>
   </link>
-  <link name="camera_link">
+  <link name="camera_base">
     <inertial>
       <mass value="0.01"/>
@@ -554,5 +554,5 @@
   <joint name="camera_joint" type="fixed">
     <parent link="base_link"/>
-    <child link="camera_link"/>
+    <child link="camera_base"/>
     <origin xyz="0.3 0 0.10" rpy="0 0 0"/>
   </joint>

Commit message: fix: imu_linkとgps_linkを正しい位置に修正

File: trc2026_description/urdf/trc2026.xacro (robot description, xacro)
@@ -408,4 +408,11 @@
     </inertial>
   </link>
+  <link name="gps_link">
+    <inertial>
+      <mass value="0.01"/>
+      <origin xyz="0 0 0" rpy="0 0 0"/>
+      <inertia ixx="1e-6" ixy="0" ixz="0" iyy="1e-6" iyz="0" izz="1e-6"/>
+    </inertial>
+  </link>
   <link name="camera_link">
     <inertial>
@@ -545,5 +552,5 @@
     <parent link="base_link"/>
     <child link="imu_link"/>
-    <origin xyz="-0.05 0 0.08" rpy="0 0 0"/>
+    <origin xyz="-0.06 0 0.03" rpy="0 0 1.57"/>
   </joint>
   <joint name="lidar_joint" type="fixed">
@@ -557,3 +564,8 @@
     <origin xyz="0.1 0 0.15" rpy="0 0 0"/>
   </joint>
+  <joint name="gps_joint" type="fixed">
+    <parent link="base_link"/>
+    <child link="gps_link"/>
+    <origin xyz="-0.35 -0.20 0.95" rpy="0 0 0"/>
+  </joint>
 </robot>

Commit message: feat: シミュレータ上でarucoミッションを再現

File: trc2026_description/urdf/trc2026.xacro (robot description, xacro)
@@ -3,4 +3,5 @@
   xmlns:xacro="http://www.ros.org/wiki/xacro">
   <xacro:arg name="use_fake_hardware"            default="false" />
+  <xacro:arg name="include_arm"                  default="true" />
   <xacro:include filename="$(find trc2026_description)/urdf/materials.xacro" />
   <xacro:include filename="$(find trc2026_description)/urdf/trc2026.trans" />
@@ -232,4 +233,5 @@
     </collision>
   </link>
+  <xacro:if value="$(arg include_arm)">
   <link name="arm_1_link">
     <inertial>
@@ -392,6 +394,19 @@
     </collision>
   </link>
-  <link name="arm_3_virtual_link"/>
-  <link name="shaft_virtual_link"/>
+  <link name="arm_3_virtual_link">
+    <inertial>
+      <mass value="0.001"/>
+      <origin xyz="0 0 0" rpy="0 0 0"/>
+      <inertia ixx="1e-6" ixy="0" ixz="0" iyy="1e-6" iyz="0" izz="1e-6"/>
+    </inertial>
+  </link>
+  <link name="shaft_virtual_link">
+    <inertial>
+      <mass value="0.001"/>
+      <origin xyz="0 0 0" rpy="0 0 0"/>
+      <inertia ixx="1e-6" ixy="0" ixz="0" iyy="1e-6" iyz="0" izz="1e-6"/>
+    </inertial>
+  </link>
+  </xacro:if>
   <link name="base_scan">
     <inertial>
@@ -482,4 +497,5 @@
     <axis xyz="-0.0 1.0 -0.0"/>
   </joint>
+  <xacro:if value="$(arg include_arm)">
   <joint name="hand_right_joint" type="prismatic">
     <origin xyz="-0.1077 -7e-06 0.082" rpy="0 0 0"/>
@@ -549,4 +565,5 @@
     <mimic joint="arm_2_joint" multiplier="-1.0" offset="0.0"/>
   </joint>
+  </xacro:if>
   <joint name="imu_joint" type="fixed">
     <parent link="base_link"/>
